File: hardware/WemosD1Mini/Kicad/SigKSens.sch (KiCad schematic (older format))
At the start: 11 parts, among them U1 LTV-824

Commit message: DC Monitor Circuit
Parts:
- added U?: ADS1115, symbol ADS1115
Connections:
- wire segments 25 -> 31
Other:
- note added: "ADS1115 Breakout board"
Changed lines of the file:
@@
 $Descr A4 11693 8268
 encoding utf-8
-Sheet 1 1
+Sheet 1 2
 Title ""
 Date ""
@@
 	1    0    0    -1
 $EndComp
-Wire Wire Line
-	4850 3600 4850 3850
-Wire Wire Line
-	4850 3950 4600 3950
 Text Label 4350 4300 3    60   ~ 0
 D7
@@
 	0    -1   -1   0
 $EndComp
-Wire Wire Line
-	3950 2800 4250 2800
-Wire Wire Line
-	3950 2600 4250 2600
-Wire Wire Line
-	1850 2800 1550 2800
 $Comp
 L R R?
@@
 	0    -1   -1   0
 $EndComp
-Wire Wire Line
-	7800 1350 8500 1350
-Wire Wire Line
-	7800 1850 8500 1850
 $Comp
 L R R?
@@
 	-1   0    0    1
 $EndComp
-Wire Wire Line
-	6900 1350 6700 1350
-Wire Wire Line
-	6700 1350 6700 1500
-Wire Wire Line
-	7200 1550 6700 1550
-Wire Wire Line
-	6700 1550 6700 1600
-Wire Wire Line
-	6900 1850 6900 1700
-Wire Wire Line
-	6900 1700 6700 1700
-Wire Wire Line
-	7200 2050 6700 2050
-Wire Wire Line
-	6700 2050 6700 1800
 Text Notes 2100 4350 0    60   ~ 0
 Config Reset button
-Wire Notes Line
-	1850 3500 1850 4450
-Wire Notes Line
-	1850 4450 3250 4450
-Wire Notes Line
-	3250 4450 3250 3500
-Wire Notes Line
-	3250 3500 1850 3500
-Wire Wire Line
-	4600 3950 4600 3600
-Wire Wire Line
-	4350 3900 4350 4300
-Wire Wire Line
-	4850 4050 4350 4050
-Connection ~ 4350 4050
-Wire Notes Line
-	4050 3350 4050 4550
-Wire Notes Line
-	4050 4550 5350 4550
-Wire Notes Line
-	5350 4550 5350 3350
-Wire Notes Line
-	5350 3350 4050 3350
 Text Notes 4750 4500 0    60   ~ 0
 1Wire Bus
 Text Notes 7150 2450 0    60   ~ 0
 2X Digital Input
-Wire Notes Line
-	6200 1100 6200 2550
-Wire Notes Line
-	6200 2550 8800 2550
-Wire Notes Line
-	8800 2550 8800 1100
-Wire Notes Line
-	8800 1100 6200 1100
 $Comp
 L MPU9255 U?
@@
 	-1   0    0    1
 $EndComp
-Wire Wire Line
-	2700 5700 3050 5700
-Wire Wire Line
-	3050 5700 3050 5600
-Wire Wire Line
-	2700 5800 3350 5800
-Wire Wire Line
-	3350 5800 3350 5600
 Text Label 3200 6400 0    60   ~ 0
 D6
-Wire Wire Line
-	2700 6400 3200 6400
 Text Label 3200 6000 0    60   ~ 0
 D2
 Text Label 3200 5900 0    60   ~ 0
 D1
-Wire Wire Line
-	2700 5900 3200 5900
-Wire Wire Line
-	2700 6000 3200 6000
 Text Notes 2000 6900 0    60   ~ 0
 MPU925X Breakout board
-Wire Notes Line
-	1650 5250 1650 7000
-Wire Notes Line
-	1650 7000 3600 7000
-Wire Notes Line
-	3600 7000 3600 5250
-Wire Notes Line
-	3600 5250 1650 5250
 $Comp
 L WemosD1Mini U?
@@
 	1    0    0    -1
 $EndComp
+$Comp
+L ADS1115 U?
+U 1 1 5A892293
+P 4250 6150
+F 0 "U?" H 4250 6050 60  0000 C CNN
+F 1 "ADS1115" H 4250 6150 60  0000 C CNN
+F 2 "" H 4250 6300 60  0001 C CNN
+F 3 "" H 4250 6300 60  0001 C CNN
+	1    4250 6150
+	1    0    0    -1
+$EndComp
+$Comp
+L +3.3V #PWR?
+U 1 1 5A8924E2
+P 4850 5550
+F 0 "#PWR?" H 4850 5400 50  0001 C CNN
+F 1 "+3.3V" H 4850 5690 50  0000 C CNN
+F 2 "" H 4850 5550 50  0001 C CNN
+F 3 "" H 4850 5550 50  0001 C CNN
+	1    4850 5550
+	1    0    0    -1
+$EndComp
+$Comp
+L GND #PWR?
+U 1 1 5A892514
+P 5050 5550
+F 0 "#PWR?" H 5050 5300 50  0001 C CNN
+F 1 "GND" H 5050 5400 50  0000 C CNN
+F 2 "" H 5050 5550 50  0001 C CNN
+F 3 "" H 5050 5550 50  0001 C CNN
+	1    5050 5550
+	-1   0    0    1
+$EndComp
+Text Label 5200 5900 0    60   ~ 0
+D1
+Text Label 5200 6000 0    60   ~ 0
+D2
+Wire Wire Line
+	4850 3600 4850 3850
+Wire Wire Line
+	4850 3950 4600 3950
+Wire Wire Line
+	3950 2800 4250 2800
+Wire Wire Line
+	3950 2600 4250 2600
+Wire Wire Line
+	1850 2800 1550 2800
+Wire Wire Line
+	7800 1350 8500 1350
+Wire Wire Line
+	7800 1850 8500 1850
+Wire Wire Line
+	6900 1350 6700 1350
+Wire Wire Line
+	6700 1350 6700 1500
+Wire Wire Line
+	7200 1550 6700 1550
+Wire Wire Line
+	6700 1550 6700 1600
+Wire Wire Line
+	6900 1850 6900 1700
+Wire Wire Line
+	6900 1700 6700 1700
+Wire Wire Line
+	7200 2050 6700 2050
+Wire Wire Line
+	6700 2050 6700 1800
+Wire Notes Line
+	1850 3500 1850 4450
+Wire Notes Line
+	1850 4450 3250 4450
+Wire Notes Line
+	3250 4450 3250 3500
+Wire Notes Line
+	3250 3500 1850 3500
+Wire Wire Line
+	4600 3950 4600 3600
+Wire Wire Line
+	4350 3900 4350 4300
+Wire Wire Line
+	4850 4050 4350 4050
+Connection ~ 4350 4050
+Wire Notes Line
+	4050 3350 4050 4550
+Wire Notes Line
+	4050 4550 5350 4550
+Wire Notes Line
+	5350 4550 5350 3350
+Wire Notes Line
+	5350 3350 4050 3350
+Wire Notes Line
+	6200 1100 6200 2550
+Wire Notes Line
+	6200 2550 8800 2550
+Wire Notes Line
+	8800 2550 8800 1100
+Wire Notes Line
+	8800 1100 6200 1100
+Wire Wire Line
+	2700 5700 3050 5700
+Wire Wire Line
+	3050 5700 3050 5600
+Wire Wire Line
+	2700 5800 3350 5800
+Wire Wire Line
+	3350 5800 3350 5600
+Wire Wire Line
+	2700 6400 3200 6400
+Wire Wire Line
+	2700 5900 3200 5900
+Wire Wire Line
+	2700 6000 3200 6000
+Wire Notes Line
+	1650 5250 1650 7000
+Wire Notes Line
+	1650 7000 3600 7000
+Wire Notes Line
+	3600 7000 3600 5250
+Wire Notes Line
+	3600 5250 1650 5250
+Wire Wire Line
+	4700 5700 4850 5700
+Wire Wire Line
+	4850 5700 4850 5550
+Wire Wire Line
+	4700 5800 5050 5800
+Wire Wire Line
+	5050 5800 5050 5550
+Wire Wire Line
+	4700 5900 5200 5900
+Wire Wire Line
+	4700 6000 5200 6000
+Wire Notes Line
+	3900 5250 3900 7000
+Wire Notes Line
+	3900 7000 5400 7000
+Wire Notes Line
+	5400 7000 5400 5250
+Wire Notes Line
+	5400 5250 3900 5250
+Text Notes 4100 6900 0    60   ~ 0
+ADS1115 Breakout board
+$Sheet
+S 7000 5250 1900 1000
+U 5A896B08
+F0 "DCMonitor" 60
+F1 "DCMonitor.sch" 60
+$EndSheet
 $EndSCHEMATC
