File: hardware/CustomESP32/Power.sch (KiCad schematic (older format))
At the start: 17 parts, among them J1 Jack-DC, U1 MP2359, U2 ME6211

Commit message: ESP32 WIP
Parts:
- added F1: Fuse, symbol Device:Fuse_Small
- R6: value 9.53k -> 9.53k 1%
- R7: value 49.9k -> 49.9k 1%
Connections:
- wire segments 42 -> 44
Other:
- moved on the sheet: R6, R7
Changed lines of the file:
@@
 L Device:R_Small R6
 U 1 1 5BAC8FF3
-P 6200 5350
-F 0 "R6" V 6304 5350 50  0000 C CNN
-F 1 "9.53k" V 6395 5350 50  0000 C CNN
-F 2 "" H 6200 5350 50  0001 C CNN
-F 3 "~" H 6200 5350 50  0001 C CNN
-	1    6200 5350
+P 6200 5500
+F 0 "R6" V 6304 5500 50  0000 C CNN
+F 1 "9.53k 1%" V 6395 5500 50  0000 C CNN
+F 2 "" H 6200 5500 50  0001 C CNN
+F 3 "~" H 6200 5500 50  0001 C CNN
+	1    6200 5500
 	-1   0    0    1
 $EndComp
@@
 L power:GND #PWR0123
 U 1 1 5BAC9068
-P 6200 5450
-F 0 "#PWR0123" H 6200 5200 50  0001 C CNN
-F 1 "GND" H 6205 5277 50  0000 C CNN
-F 2 "" H 6200 5450 50  0001 C CNN
-F 3 "" H 6200 5450 50  0001 C CNN
-	1    6200 5450
+P 6200 5600
+F 0 "#PWR0123" H 6200 5350 50  0001 C CNN
+F 1 "GND" H 6205 5427 50  0000 C CNN
+F 2 "" H 6200 5600 50  0001 C CNN
+F 3 "" H 6200 5600 50  0001 C CNN
+	1    6200 5600
 	1    0    0    -1
 $EndComp
@@
 $EndComp
 Wire Wire Line
-	6000 5150 6200 5150
-Wire Wire Line
-	6200 5150 6200 5250
+	6200 5150 6200 5400
 $Comp
 L Device:R_Small R7
 U 1 1 5BAC9ACA
-P 6400 5150
-F 0 "R7" V 6296 5150 50  0000 C CNN
-F 1 "49.9k" V 6205 5150 50  0000 C CNN
-F 2 "" H 6400 5150 50  0001 C CNN
-F 3 "~" H 6400 5150 50  0001 C CNN
-	1    6400 5150
+P 6700 5150
+F 0 "R7" V 6596 5150 50  0000 C CNN
+F 1 "49.9k 1%" V 6505 5150 50  0000 C CNN
+F 2 "" H 6700 5150 50  0001 C CNN
+F 3 "~" H 6700 5150 50  0001 C CNN
+	1    6700 5150
 	0    -1   -1   0
 $EndComp
-Connection ~ 6200 5150
 Wire Wire Line
-	6200 5150 6300 5150
-Wire Wire Line
-	6500 5150 7500 5150
+	6800 5150 7500 5150
 Connection ~ 7500 5150
 Wire Wire Line
@@
 L power:+BATT #PWR0127
 U 1 1 5BAD7730
-P 2050 4800
-F 0 "#PWR0127" H 2050 4650 50  0001 C CNN
-F 1 "+BATT" V 2065 4928 50  0000 L CNN
-F 2 "" H 2050 4800 50  0001 C CNN
-F 3 "" H 2050 4800 50  0001 C CNN
-	1    2050 4800
+P 2900 4800
+F 0 "#PWR0127" H 2900 4650 50  0001 C CNN
+F 1 "+BATT" V 2915 4928 50  0000 L CNN
+F 2 "" H 2900 4800 50  0001 C CNN
+F 3 "" H 2900 4800 50  0001 C CNN
+	1    2900 4800
 	0    1    1    0
 $EndComp
+$Comp
+L Device:Fuse_Small F1
+U 1 1 5BB2CFE8
+P 2400 4800
+F 0 "F1" H 2400 4985 50  0000 C CNN
+F 1 "Fuse" H 2400 4894 50  0000 C CNN
+F 2 "" H 2400 4800 50  0001 C CNN
+F 3 "~" H 2400 4800 50  0001 C CNN
+	1    2400 4800
+	1    0    0    -1
+$EndComp
+Wire Wire Line
+	2050 4800 2300 4800
+Wire Wire Line
+	2500 4800 2900 4800
+Wire Wire Line
+	6000 5150 6200 5150
+Connection ~ 6200 5150
+Wire Wire Line
+	6200 5150 6600 5150
 $EndSCHEMATC
