File: hardware/CustomESP32/ESP32 Windlass.sch (KiCad schematic (older format))
At the start: 58 parts, among them J1 Conn_01x06, J2 Screw_Terminal_01x06, K1 RESET, U1 BTS7004-1EPP, U2 BTS7004-1EPP, U3 ESP32-WROVER, U4 ADS1015IDGS, U5 LM5166Y

Commit message: some updates to pcb
Other:
- note added: "need cap"
- note added: "needs polarity!"
Changed lines of the file:
@@
 Text Notes 2300 1950 0    50   ~ 0
 INPUT Only :(
+Text Notes 2500 7100 0    50   ~ 0
+needs polarity!
+Text Notes 6600 4950 0    50   ~ 0
+need cap
 $EndSCHEMATC
